Commit message: [data][launch](3.12) Fix and Modifify Launch files and assosiated xml files in data directory

File: data/includes/urdf/Turtlebot_Kinect_Lidar.urdf.xacro (robot description, xacro)
@@ -6,5 +6,5 @@
        xmlns:xacro="http://ros.org/wiki/xacro">
   <!-- Defines the kobuki component tag. -->
-  <xacro:include filename="$(find ecobot)/launch/includes/urdf/kobuki.urdf.xacro" />
+  <xacro:include filename="$(find ecobot)/data/includes/urdf/kobuki.urdf.xacro" />
   <xacro:include filename="$(find turtlebot_description)/urdf/stacks/hexagons.urdf.xacro"/>
   <xacro:include filename="$(find turtlebot_description)/urdf/sensors/kinect.urdf.xacro"/><kobuki/>

File: data/includes/urdf/kobuki.urdf.xacro (robot description, xacro)
@@ -7,6 +7,6 @@
  -->
 <robot name="kobuki" xmlns:xacro="http://ros.org/wiki/xacro">
-  <xacro:include filename="$(find ecobot)/launch/includes/urdf/common_properties.urdf.xacro"/>
-  <xacro:include filename="$(find ecobot)/launch/includes/urdf/kobuki_gazebo.urdf.xacro"/>
+  <xacro:include filename="$(find ecobot)/data/includes/urdf/common_properties.urdf.xacro"/>
+  <xacro:include filename="$(find ecobot)/data/includes/urdf/kobuki_gazebo.urdf.xacro"/>
   <!-- Kobuki -->
   <xacro:macro name="kobuki">
@@ -30,5 +30,5 @@
         <geometry>
           <!-- new mesh -->
-          <mesh filename="package://ecobot/launch/includes/meshes/main_body.dae" />
+          <mesh filename="package://ecobot/data/includes/meshes/main_body.dae" />
         </geometry>
         <origin xyz="0.001 0 0.05199" rpy="0 0 0"/>
@@ -65,5 +65,5 @@
       <visual>
         <geometry>
-          <mesh filename="package://ecobot/launch/includes/meshes/wheel.dae"/>
+          <mesh filename="package://ecobot/data/includes/meshes/wheel.dae"/>
         </geometry>
         <origin xyz="0 0 0" rpy="0 0 0"/>
@@ -92,5 +92,5 @@
       <visual>
         <geometry>
-          <mesh filename="package://ecobot/launch/includes/meshes/wheel.dae"/>
+          <mesh filename="package://ecobot/data/includes/meshes/wheel.dae"/>
         </geometry>
         <origin xyz="0 0 0" rpy="0 0 0"/>
@@ -223,5 +223,5 @@
       <origin xyz="0 0 0" rpy="0 0 0"/>
       <geometry>
-        <mesh filename="package://ecobot/launch/includes/meshes/hokuyo.dae"/>
+        <mesh filename="package://ecobot/data/includes/meshes/hokuyo.dae"/>
       </geometry>
     </visual>
